File: designing/codec_AD1938/Hardware/DAC_buffer_non-inv.brd (EAGLE design)
At the start: 100 x 80 mm, 25 parts, among them IC1 TL072D

Commit message: Dev folder added
Parts:
- moved C13 110.7 mm to (26.1, 31.1), turned to 180 degrees
- moved C14 94.7 mm to (14.6, 29.8), turned to 180 degrees
- moved R12 59.1 mm to (22.9, 27.9)
- moved R14 56.0 mm to (15.2, 32.4)
- moved R13 52.1 mm to (15.2, 25.4), turned to 180 degrees
- moved R11 49.1 mm to (19.1, 27.9), turned to 180 degrees
- moved C11 48.3 mm to (22.9, 24.1)
- moved R10 47.0 mm to (22.9, 26.0)
- moved C12 39.4 mm to (15.2, 27.3), turned to 180 degrees
- moved R9 37.8 mm to (19.1, 24.1)
- moved C10 37.1 mm to (19.1, 26.0), turned to 180 degrees
- moved R8 31.1 mm to (15.2, 34.3)
- moved C9 15.9 mm to (14.6, 36.8)
- moved C6 10.3 mm to (22.9, 42.5), turned to 0 degrees
- moved C7 9.25 mm to (15.2, 39.4)
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